Commit message: grg

File: src/perseus_arm/robot.urdf (robot description, URDF)
Before this commit: robot my-robot-urdf, 14 links, 13 joints
Joints:
- joint base: limit lower=-3.141592653589793 upper=3.141592653589793 effort=10 velocity=10 -> lower=-1.570796 upper=1.570796 effort=10 velocity=10
- joint elbow: limit lower=-3.141592653589793 upper=3.141592653589793 effort=10 velocity=10 -> lower=-1.570796 upper=1.570796 effort=10 velocity=10
- joint shoulder: limit lower=-3.141592653589793 upper=3.141592653589793 effort=10 velocity=10 -> lower=-1.570796 upper=1.570796 effort=10 velocity=10
